File: pcb/usb_auto_reboot.kicad_pcb (KiCad board)
At the start: 2 copper layers, 14.2 x 26 mm, 11 parts, among them J1 USB2.0 C 12Pin Receptable, J2 USB3.0 C Plug, U1 CH217K, U2 CH32V003J4M6

Commit message: update README
Changed lines of the file:
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@@
     (fp_line (start 1 0.6) (end 1 -0.6)
       (stroke (width 0.1) (type solid)) (layer "F.Fab"))
-    (pad "1" smd roundrect (at -1.025 0) (size 1.15 1.4) (layers "F.Cu" "F.Paste" "F.Mask") (roundrect_rratio 0.2173913043)
+    (pad "1" smd roundrect (at -1.025 0) (size 1.15 1.4) (layers "F.Cu" "F.Paste" "F.Mask") (roundrect_rratio 0.217391)
       (net 2 "GND") (pinfunction "K") (pintype "passive"))
-    (pad "2" smd roundrect (at 1.025 0) (size 1.15 1.4) (layers "F.Cu" "F.Paste" "F.Mask") (roundrect_rratio 0.2173913043)
+    (pad "2" smd roundrect (at 1.025 0) (size 1.15 1.4) (layers "F.Cu" "F.Paste" "F.Mask") (roundrect_rratio 0.217391)
       (net 5 "Net-(D1-A)") (pinfunction "A") (pintype "passive"))
     (model "${KICAD6_3DMODEL_DIR}/LED_SMD.3dshapes/LED_0805_2012Metric.wrl"
@@
     (pad "12" smd rect (at 3.2 -7.525) (size 0.6 1.15) (layers "F.Cu" "F.Paste" "F.Mask")
       (net 2 "GND") (pinfunction "GND_A12/B1") (pintype "power_out"))
-    (model "/Users/nnyn/ghq/github.com/74th/my-kicad-parts/footprints/USB-C-12-Pin-MidMount.step"
-      (offset (xyz 0 -0.2 0))
-      (scale (xyz 1 1 1))
-      (rotate (xyz 90 180 180))
+    (model "/Users/nnyn/ghq/github.com/74th/my-kicad-parts/footprints/USB-C-12-Pin-MidMount,Molex,2169900002.stp"
+      (offset (xyz 0 3.8 1.2))
+      (scale (xyz 1 1 1))
+      (rotate (xyz 90 180 0))
     )
   )
@@
     (fp_rect (start -1.88 -0.98) (end 1.88 0.98)
       (stroke (width 0.05) (type default)) (fill none) (layer "F.CrtYd"))
-    (pad "1" smd roundrect (at -1 0 90) (size 1.2 1.4) (layers "F.Cu" "F.Paste" "F.Mask") (roundrect_rratio 0.2083333333)
+    (pad "1" smd roundrect (at -1 0 90) (size 1.2 1.4) (layers "F.Cu" "F.Paste" "F.Mask") (roundrect_rratio 0.208333)
       (net 14 "Net-(U1-ISET)") (pintype "passive"))
-    (pad "2" smd roundrect (at 1 0 90) (size 1.2 1.4) (layers "F.Cu" "F.Paste" "F.Mask") (roundrect_rratio 0.2083333333)
+    (pad "2" smd roundrect (at 1 0 90) (size 1.2 1.4) (layers "F.Cu" "F.Paste" "F.Mask") (roundrect_rratio 0.208333)
       (net 2 "GND") (pintype "passive"))
     (model "${KICAD6_3DMODEL_DIR}/Resistor_SMD.3dshapes/R_0805_2012Metric.wrl"
@@
     (fp_rect (start -1.88 0.98) (end 1.88 -0.98)
       (stroke (width 0.05) (type default)) (fill none) (layer "B.CrtYd"))
-    (pad "1" smd roundrect (at -1.0375 0 90) (size 1.175 1.45) (layers "B.Cu" "B.Paste" "B.Mask") (roundrect_rratio 0.2127659574)
+    (pad "1" smd roundrect (at -1.0375 0 90) (size 1.175 1.45) (layers "B.Cu" "B.Paste" "B.Mask") (roundrect_rratio 0.212766)
       (net 1 "+5V") (pintype "passive"))
-    (pad "2" smd roundrect (at 1.0375 0 90) (size 1.175 1.45) (layers "B.Cu" "B.Paste" "B.Mask") (roundrect_rratio 0.2127659574)
+    (pad "2" smd roundrect (at 1.0375 0 90) (size 1.175 1.45) (layers "B.Cu" "B.Paste" "B.Mask") (roundrect_rratio 0.212766)
       (net 2 "GND") (pintype "passive"))
     (model "${KICAD6_3DMODEL_DIR}/Capacitor_SMD.3dshapes/C_0805_2012Metric.wrl"
@@
     (fp_rect (start -1.88 0.98) (end 1.88 -0.98)
       (stroke (width 0.05) (type default)) (fill none) (layer "B.CrtYd"))
-    (pad "1" smd roundrect (at -1.0375 0 90) (size 1.175 1.45) (layers "B.Cu" "B.Paste" "B.Mask") (roundrect_rratio 0.2127659574)
+    (pad "1" smd roundrect (at -1.0375 0 90) (size 1.175 1.45) (layers "B.Cu" "B.Paste" "B.Mask") (roundrect_rratio 0.212766)
       (net 1 "+5V") (pintype "passive"))
-    (pad "2" smd roundrect (at 1.0375 0 90) (size 1.175 1.45) (layers "B.Cu" "B.Paste" "B.Mask") (roundrect_rratio 0.2127659574)
+    (pad "2" smd roundrect (at 1.0375 0 90) (size 1.175 1.45) (layers "B.Cu" "B.Paste" "B.Mask") (roundrect_rratio 0.212766)
       (net 2 "GND") (pintype "passive"))
     (model "${KICAD6_3DMODEL_DIR}/Capacitor_SMD.3dshapes/C_0805_2012Metric.wrl"
@@
     (fp_rect (start -1.88 0.98) (end 1.88 -0.98)
       (stroke (width 0.05) (type default)) (fill none) (layer "B.CrtYd"))
-    (pad "1" smd roundrect (at -1 0 270) (size 1.2 1.4) (layers "B.Cu" "B.Paste" "B.Mask") (roundrect_rratio 0.2083333333)
+    (pad "1" smd roundrect (at -1 0 270) (size 1.2 1.4) (layers "B.Cu" "B.Paste" "B.Mask") (roundrect_rratio 0.208333)
       (net 15 "/LED") (pintype "passive"))
-    (pad "2" smd roundrect (at 1 0 270) (size 1.2 1.4) (layers "B.Cu" "B.Paste" "B.Mask") (roundrect_rratio 0.2083333333)
+    (pad "2" smd roundrect (at 1 0 270) (size 1.2 1.4) (layers "B.Cu" "B.Paste" "B.Mask") (roundrect_rratio 0.208333)
       (net 5 "Net-(D1-A)") (pintype "passive"))
     (model "${KICAD6_3DMODEL_DIR}/Resistor_SMD.3dshapes/R_0805_2012Metric.wrl"
