File: pcb/usb_auto_reboot.kicad_sch (KiCad schematic)
At the start: 11 parts, among them J1 USB2.0 C 12Pin Receptable, J2 USB3.0 C Plug, U1 CH217K, U2 CH32V003J4M6

Commit message: update README
Parts:
- J1: value USB2.0 C 12Pin Receptable -> GCT USB4510-03-1-A
Changed lines of the file:
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@@
       (effects (font (size 1.27 1.27)))
     )
-    (property "Value" "USB2.0 C 12Pin Receptable" (at 70.485 39.37 0)
+    (property "Value" "GCT USB4510-03-1-A" (at 70.485 39.37 0)
       (effects (font (size 1.27 1.27)))
     )
